Commit message: switched to ros2

File: racecar_description/urdf/racecar.xacro (robot description, xacro)
@@ -46,5 +46,5 @@
     <visual>
       <xacro:left_rear_wheel_geometry />
-      <material name="black" />
+      <material name="Black" />
     </visual>
     <collision>robot
@@ -67,5 +67,5 @@
     <visual>
       <xacro:right_rear_wheel_geometry />
-      <material name="black" />
+      <material name="Black" />
     </visual>
     <collision>
@@ -88,5 +88,5 @@
     <visual>
       <xacro:left_steering_hinge_geometry />
-      <material name="grey" />
+      <material name="DarkGrey" />
     </visual>
   </link>
@@ -106,5 +106,5 @@
     <visual>
       <xacro:right_steering_hinge_geometry />
-      <material name="grey" />
+      <material name="DarkGrey" />
     </visual>
   </link>
@@ -124,5 +124,5 @@
     <visual>
       <xacro:left_front_wheel_geometry />
-      <material name="black" />
+      <material name="Black" />
     </visual>
     <collision>
@@ -145,5 +145,5 @@
     <visual>
       <xacro:right_front_wheel_geometry />
-      <material name="black" />
+      <material name="Black" />
     </visual>
     <collision>
@@ -174,5 +174,5 @@
       <geometry>
         <mesh filename="package://racecar_description/meshes/hokuyo.dae"/>
-        <material name="grey" />
+        <material name="DarkGrey" />
       </geometry>
     </visual>
@@ -202,5 +202,5 @@
         <box size="0.033 0.03 0.030"/>
       </geometry>
-      <material name="red"/>
+      <material name="Red"/>
     </visual>
   </link>

Commit message: fix imu urdf

File: racecar_description/urdf/racecar.xacro (robot description, xacro)
@@ -225,9 +225,4 @@
   </joint>
   <!-- IMU -->
-  <joint name="imu_joint" type="fixed">
-    <origin xyz="0 -0.065 -0.015" rpy="0 0 -1.570796327" />
-    <parent link="$(arg prefix)/base_laser"/>
-    <child link="$(arg prefix)/imu_link" />
-  </joint>
   <link name='$(arg prefix)/imu_link'>
      <inertial>
@@ -240,4 +235,9 @@
        </inertial>
   </link>
+  <joint name="imu_joint" type="fixed">
+    <origin xyz="0.3 -0.115 0" rpy="${pi} 0 0" />
+    <parent link="$(arg prefix)/base_link"/>
+    <child link="$(arg prefix)/imu_link" />
+  </joint>
   <!-- Add the remaining xacros -->
   <xacro:include filename="$(find racecar_description)/urdf/racecar.gazebo"/>

Commit message: fix frame and remove unused file

File: racecar_description/urdf/racecar.xacro (robot description, xacro)
@@ -236,5 +236,5 @@
   </link>
   <joint name="imu_joint" type="fixed">
-    <origin xyz="0.3 -0.115 0" rpy="${pi} 0 0" />
+    <origin xyz="0.3 -0.115 0" rpy="0 0 0" />
     <parent link="$(arg prefix)/base_link"/>
     <child link="$(arg prefix)/imu_link" />
